Commit message: flipped and added joint

File: robot_description/urdf/robot.urdf (robot description, URDF)
Before this commit: robot my_robot, 3 links, 2 joints
Links:
- added link second_link, mass 1; collision mesh filename=package://robot_simulation/robot_description/meshes/link.STL scale=0.001 0.001 0.001; visual mesh filename=package://robot_simulation/robot_description/meshes/link.STL scale=0.001 0.001 0.001
- link first_link: geometry collision mesh filename=package://robot_simulation/robot_description/meshes/link.STL scale=0.001 0.001 0.001; visual mesh filename=package://robot_simulation/robot_description/meshes/link.STL scale=0.001 0.001 0.001
Joints:
- added joint first_to_second_joint: type continuous, parent first_link, child second_link, origin xyz=0 0 0.5 rpy=0 0 0, axis 0 1 0
- joint base_to_first_joint: axis (none) -> 0 1 0; origin xyz=0 0 0.130 rpy=0 0 0 -> xyz=0 0 0.06 rpy=0 0.785 0
- joint fixed: origin (none) -> xyz=0 0 1.25 rpy=3.14159 0 0

Commit message: two link with controllers and torque limits

File: robot_description/urdf/robot.urdf (robot description, URDF)
Before this commit: robot my_robot, 4 links, 3 joints
Links:
- link first_link: mass 1 -> 0.15156
- link second_link: mass 1 -> 0.15156
Joints:
- joint base_to_first_joint: limit (none) -> effort=1.0 velocity=30.0
- joint first_to_second_joint: limit (none) -> effort=1.0 velocity=30.0

Commit message: new stuff

File: robot_description/urdf/robot.urdf (robot description, URDF)
Before this commit: robot my_robot, 4 links, 3 joints
Links:
- added link end_effector_latch_link, mass 2.745e-3; collision mesh filename=package://robot_simulation/robot_description/meshes/end_eff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 scale=0.001 0.001 0.001; visual mesh filename=package://robot_simulation/robot_description/meshes/end_eff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 scale=0.001 0.001 0.001
- added link end_effector_link, mass 0.03233; collision mesh filename=package://robot_simulation/robot_description/meshes/end_eff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 scale=0.001 0.001 0.001; visual mesh filename=package://robot_simulation/robot_description/meshes/end_eff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 scale=0.001 0.001 0.001
- link first_link: mass 0.15156 -> 0.05028; geometry collision mesh filename=package://robot_simulation/robot_description/meshes/first_l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 scale=0.001 0.001 0.001; visual mesh filename=package://robot_simulation/robot_description/meshes/first_l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 scale=0.001 0.001 0.001
- link second_link: mass 0.15156 -> 0.04670; geometry collision mesh filename=package://robot_simulation/robot_description/meshes/second_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 scale=0.001 0.001 0.001; visual mesh filename=package://robot_simulation/robot_description/meshes/second_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 scale=0.001 0.001 0.001
Joints:
- removed joint fixed
- added joint base_link_joint: type continuous, parent world, child base_link, origin xyz=0 0 1.25 rpy=3.14159 0 0, axis 0 0 1
- added joint end_effector_to_latch: type continuous, parent end_effector_link, child end_effector_latch_link, origin xyz=0.0125 0 -0.01 rpy= -1.570796 -1.470796 0, axis 0 0 1, limit effort=1.0 velocity=30.0
- added joint second_to_end_effector: type fixed, parent second_link, child end_effector_link, origin xyz=0 0 0.3 rpy=0 0 0, axis 0 1 0, limit effort=1.0 velocity=30.0
- joint base_to_first_joint: origin xyz=0 0 0.06 rpy=0 0.785 0 -> xyz=0 0 0.06 rpy=0 0 0
- joint first_to_second_joint: origin xyz=0 0 0.5 rpy=0 0 0 -> xyz=0 0 0.3 rpy=0 0 0

Commit message: new stuff

File: robot_description/urdf/robot.urdf (robot description, URDF)
Before this commit: robot my_robot, 6 links, 5 joints
Joints:
- joint base_link_joint: origin xyz=0 0 1.25 rpy=3.14159 0 0 -> xyz=0 0 1.0 rpy=3.14159 0 0
- joint base_to_first_joint: limit effort=1.0 velocity=30.0 -> effort=5.0 velocity=30.0
- joint first_to_second_joint: limit effort=1.0 velocity=30.0 -> effort=3.0 velocity=30.0

File: target_description/urdf/projectile.urdf (robot description, URDF)
Before this commit: robot my_projectile, 2 links, 1 joints
Joints:
- joint projectile_joint: origin xyz=0.005 0 0.565 rpy=0 0 0 -> xyz=0.005 0 0.315 rpy=0 0 0

File: target_description/urdf/target.urdf (robot description, URDF)
Before this commit: robot my_target, 2 links, 1 joints
Joints:
- joint fixed: origin xyz=5 0 0 rpy=0 0 0 -> xyz=3 0 0 rpy=0 0 0
